File: hardware/pcb/Board_2_Eagle/Board_2.sch (EAGLE design)
At the start: 75 parts, among them IC1 MCP73831, IC2 LT1963EST-1.5, IC3 VUB300, IC30 TS3A27, IC4 ISP1507, IC5 WTV020SD-20S, J3 DEBUG_CONNECTOR, SW1 SW_TACT_SMD, SW2 SW_TACT_SMD, SW3 SW_TACT_SMD, SW4 SW_TACT_SMD, SW5 SW_TACT_SMD, U1 PAM8302AASCR, X1 1751248, X2 1751248, X3 1751248, X4 1751248, X5 1751248, Y1 CRYSTAL.3.2X2.5MM

Commit message: huhu
Parts:
- C29: value 0R -> 10u
- C34: value 100u -> 100u Tan
- R8, R9: value Ferit Bead -> 0R
- T1, T3: value (none) -> IRLML6302TRPBF
- T2: value (none) -> 1HP04CH
Other:
- note added: "/EN"
- note added: "0"
- note added: "1"
- note added: "IN"
- note added: "Kondensator verhindert, dass Gleichstrom durch den Knochenschallgeber fliesst."
- note added: "PWR"
- note added: "VUB_SD_PWR"
- note added: "X"
- moved on the sheet: C1, C11, C14, C15, C16, C19, C2, C20, C21, C22, C3, C34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
